File: BATAUS/BATAUS.kicad_pcb (KiCad board)
At the start: 2 copper layers, 9 parts, among them J1 Servo, J2 Screw_Terminal_01x02, J3 Screw_Terminal_01x02, K1 SRA-05VDC-CL, Q1 MMBT2222A, U1 LM7805_TO220, U3 ESP32-C3-DevKitM-1

Commit message: Correccion de errores
Parts:
- removed J1: Servo, Connector_PinHeader_2.00mm:PinHeader_1x03_P2.00mm_Vertical
- removed U3: ESP32-C3-DevKitM-1, Huellas:ESP32-S3-SuperMini
- added R1: R330, Resistor_THT:R_Axial_DIN0207_L6.3mm_D2.5mm_P10.16mm_Horizontal, F.Cu at (133.0, 69.9)
- added R4: R330, Resistor_THT:R_Axial_DIN0207_L6.3mm_D2.5mm_P10.16mm_Horizontal, F.Cu at (129.0, 69.9)
- added SW1: SW_Push, Connector_PinHeader_2.00mm:PinHeader_1x02_P2.00mm_Vertical, F.Cu at (131.0, 86.0)
- added SW2: SW_Push, Connector_PinHeader_2.00mm:PinHeader_1x02_P2.00mm_Vertical, F.Cu at (122.0, 80.0)
- added U4: ESP32-C3_SUPERMINI_TH, ESP32-C3_SUPERMINI_TH:MODULE_ESP32-C3_SUPERMINI_TH, F.Cu at (117.0, 64.5)
- R2: footprint Resistor_SMD:R_0805_2012Metric_Pad1.20x1.40mm_HandSolder -> Resistor_THT:R_Axial_DIN0207_L6.3mm_D2.5mm_P10.16mm_Horizontal; moved to F.Cu
- moved R2 12.3 mm to (94.9, 56.0), turned to 0 degrees
- moved U1 8.30 mm to (137.8, 54.5), turned to 180 degrees
- moved J3 5.81 mm to (132.8, 63.0), turned to 0 degrees
- moved J2 4.30 mm to (92.0, 83.5), turned to 0 degrees
Connections:
- D1 pad 1: Net-(D1-K) -> 5V
- K1 pad COIL1: Net-(D1-K) -> 5V
- K1 pad COM: Net-(J2-Pin_2) -> Net-(J2-Pin_1)
- K1 pad NC: Net-(J2-Pin_1) -> unconnected-(K1-PadNC)
- K1 pad NO: unconnected-(K1-PadNO) -> Net-(J2-Pin_2)
Routing:
- net LvW: track 0.00 -> 51.0 mm
- net 5V: track 10.6 -> 54.8 mm
- net LvW2: track 0.00 -> 20.8 mm
- net 3.3V: track 0.00 -> 17.8 mm
- net Net-(D1-A): track 3.15 -> 19.5 mm
- net Net-(J2-Pin_1): track 21.7 -> 13.8 mm
- net SRV: track 6.83 -> 0.00 mm
- net Net-(R1-Pad2): track 0.00 -> 5.92 mm
- net Net-(D1-K): track 5.33 -> 0.00 mm
- net DatIN1: track 9.83 -> 4.77 mm
- net Net-(Q1-B): track 4.54 -> 9.59 mm
- net Net-(R4-Pad2): track 0.00 -> 5.03 mm
- net Net-(J2-Pin_2): track 13.5 -> 14.9 mm
