File: BATAUS/BATAUS.kicad_sch (KiCad schematic)
At the start: 9 parts, among them J1 Servo, J2 Screw_Terminal_01x02, J3 Screw_Terminal_01x02, K1 SRA-05VDC-CL, Q1 MMBT2222A, U1 LM7805_TO220, U3 ESP32-C3-DevKitM-1

Commit message: Correccion de errores
Parts:
- removed J1: Servo, Connector_PinHeader_2.00mm:PinHeader_1x03_P2.00mm_Vertical, symbol Connector_Generic:Conn_01x03
- removed U3: ESP32-C3-DevKitM-1, Huellas:ESP32-S3-SuperMini, symbol RF_Module:ESP32-C3-DevKitM-1
- added R1, R4: R330, Resistor_THT:R_Axial_DIN0207_L6.3mm_D2.5mm_P10.16mm_Horizontal, symbol Device:R
- added R3, R5: R10k, symbol Device:R
- added SW1, SW2: SW_Push, Connector_PinHeader_2.00mm:PinHeader_1x02_P2.00mm_Vertical, symbol EESTN5:SW_Push
- added U4: ESP32-C3_SUPERMINI_TH, ESP32-C3_SUPERMINI_TH:MODULE_ESP32-C3_SUPERMINI_TH, symbol ESP32-C3_SUPERMINI_TH:ESP32-C3_SUPERMINI_TH
- R2: footprint Resistor_SMD:R_0805_2012Metric_Pad1.20x1.40mm_HandSolder -> Resistor_THT:R_Axial_DIN0207_L6.3mm_D2.5mm_P10.16mm_Horizontal
Connections:
- net 5V: now also D1.1 (K), K1.COIL1, U4.5V
- net DatIN1: now also U4.6 (GPIO6)
- net GND: now also R3.2, R5.2, U4.G (GND)
- net at K1.COM: now also J2.1 (Pin_1); no longer J2.2 (Pin_2)
- net at K1.NC: no longer J2.1 (Pin_1)
- net at K1.NO: now also J2.2 (Pin_2)
- new net: R4.2, SW2.2
- new net: R1.2, SW1.2
- new net 3.3V: R1.1, R4.1, U4.3.3 (3V3)
- new net LvW: R3.1, SW1.1, U4.5 (GPIO5)
- new net LvW2: R5.1, SW2.1, U4.4 (GPIO4)
Other:
- moved on the sheet: J2, J3
